File: PCB/LibreServo-v2.3.1.sch (EAGLE design)
At the start: 83 parts, among them M1 M1, M2 MOSFET_N+P, M3 MOSFET_N+P, M4 FAN3227/4, M5 FAN3227/4, U1 STM32F301/2, U10 AEAT-8800, U2 MPM3610, U3 AP2112, U4 ACS711, U5 SIT3485

Commit message: Wire MCU/RS-485 swap and CAN-FD addition into the schematic
Executes the decisions from PCB/RS485-CANFD-TPM-upgrade.md at the
netlist level in PCB/LibreServo-v2.3.1.sch:

- U1: STM32F302K8U6 -> STM32G431. Every existing net is re-pinned onto
  the G431's actual UFQFPN32 pinout (verified against the datasheet's
  alternate-function table, not assumed to match the old part).
  PA11/PA12 are the only FDCAN1-capable pins on this package, so the
  PWM-2/PWM-4 signals that used to live there move to PB3/PB4, which
  were already unused (NC-marked) on the F302 - a like-for-like swap
  with no pin-budget shortfall.
- U5: SIT3485 -> ADM2587E isolated RS-485 transceiver, wired
  half-duplex (Y+A / Z+B tied) onto the existing RS485_P/RS485_N
  daisy-chain nets, with the datasheet's isoPower support components
  added on a dedicated, deliberately-isolated ground net that has no
  connection back to board GND.
- U6 (new): ADM3055E isolated CAN-FD transceiver, TXD/RXD wired to
  U1's new FDCAN1 pins, isoPower support components on their own
  isolated ground net, CANH/CANL brought out as labeled but
  unterminated nets pending a bus-connector decision.

New devicesets for STM32G431/ADM2587E/ADM3055E are symbol-only
placeholders (no footprint yet), matching this library's existing
GND/+3V3 supply-symbol pattern - footprints, .brd placement, and the
firmware pin/timer port are still open, tracked in the updated
engineering notes doc along with a flagged gap: the ADM3055E's VCC
needs a 5V rail this board doesn't currently generate.

Co-Authored-By: Claude Sonnet 5 <noreply@anthropic.com>
Claude-Session: https://claude.ai/code/session_012wYcYVnHvvmMdDYKgLHq3u
Parts:
- removed U$12, U$13: NC_MARKER, NC_MARKER:NC_MARKER
- added B4, B5, B6: (no value), Propio:FERRITE_BEAD_0603
- added C25, C28, C29, C31, C34, C38: 100n, Propio:C-EU0402
- added C26, C27, C32, C36: 10u, Propio:C-EU0603
- added C30, C33, C37: 10n, Propio:C-EU0402
- added C35: 220n, Propio:C-EU0402
- added U$24, U$25: NC_MARKER, NC_MARKER:NC_MARKER
- added U6: ADM3055E, Propio:ADM3055E
- U1: value STM32F301/2 -> STM32G431K6/K8; device Propio:STM32F302 -> Propio:STM32G431
- U5: value SIT3485 -> ADM2587E; device Propio:RS485-HALF_DUPLEX -> Propio:ADM2587E
Connections:
- removed net N$7: U$12.P$1, U1.PB4
- removed net N$8: U$13.P$1, U1.PB3
- new net +5V_ISO_CANFD: C31.1, C32.1, U6.VCC
- new net CANFD_GNDISO: B5.1, U6.GNDISO
- new net CANFD_ISO_GND: B5.2, C35.2, C36.2, C37.2, C38.2, U6.GND2, U6.RS
- new net CANFD_VISOIN: B6.2, C37.1, C38.1, U6.VISOIN
- new net CANFD_VISOOUT: B6.1, C35.1, C36.1, U6.VISOOUT
- new net CANH: U6.CANH
- new net CANL: U6.CANL
- new net FDCAN1_RX: U1.PA11, U6.RXD
- new net FDCAN1_TX: U1.PA12, U6.TXD
- new net N$20: U$24.P$1, U6.AUXIN
- new net N$21: U$25.P$1, U6.AUXOUT
- new net RS485_ISO_GND: C27.2, C28.2, C29.2, C30.2, U5.GND2
- new net RS485_VISOIN: B4.2, C29.1, C30.1, U5.VISOIN
- new net RS485_VISOOUT: B4.1, C27.1, C28.1, U5.VISOOUT
- net +3V3: now also C25.1, C26.1, C33.1, C34.1, U5.VCC, U6.VIO; no longer U5.P$8
- net CLK-8MHZ: now also U1.PF0-OSC_IN; no longer U1.PF0/OSC_IN
- net GND: now also C25.2, C26.2, C31.2, C32.2, C33.2, C34.2, U1.PB8-BOOT0, U1.VSSA, U5.GND1, U6.GND1, U6.SILENT, U6.STBY; no longer U1.BOOT0, U1.VSSA/VREF-, U5.P$5
- net N$10: now also U1.PF1-OSC_OUT; no longer U1.PF1/OSC_OUT
- net N$11: now also U1.PG10-NRST; no longer U1.NRST
- net PWM-2: now also U1.PB4; no longer U1.PA11
- net PWM-4: now also U1.PB3; no longer U1.PA12
- net RS485_N: now also U5.B, U5.Z; no longer U5.P$7
- net RS485_P: now also U5.A, U5.Y; no longer U5.P$6
- net SEL_SERIAL: now also U5.DE, U5.RE; no longer U5.P$2, U5.P$3
- net USART1_RX: now also U5.RxD; no longer U5.P$1
- net USART1_TX: now also U5.TxD; no longer U5.P$4
Other:
- note added: "ADM2587E @ ISOLATED RS485"
- note added: "ADM3055E @ ISOLATED CAN-FD (new)"
- note added: "NEEDS: footprint/package, board placement, CANH/CANL bus connector, and a new 5V regulator for VCC (+5V_ISO_CANFD net) -- board has no 5V rail today. See PCB/RS485-CANFD-TPM-upgrade.md."
- note added: "STM32G431K6/K8 @ up to 170MHz"
- note removed: "SIT3485 @ RS485"
- note removed: "STM32F301K8 @ 72MHz"
