File: PCB/LibreServo-v2.3.1.sch (EAGLE design)
At the start: 101 parts, among them M1 M1, M2 MOSFET_N+P, M3 MOSFET_N+P, M4 FAN3227/4, M5 FAN3227/4, U1 STM32G431K6/K8, U10 AEAT-8800, U2 MPM3610, U3 AP2112, U4 ACS711, U5 ADM2587E, U6 ADM3055E

Commit message: Wire TPM (SLB9672) into the schematic as U7
Adds the SLB9672 deviceset (symbol-only placeholder, same pattern as
STM32G431/ADM2587E/ADM3055E) and instantiates it as U7, closing out the
one item the previous MCU/RS-485/CAN-FD pass deliberately left open.

A full pin-budget audit of U1 (STM32G431, UFQFPN32) found the package
fully committed after the FDCAN1 re-pin: every SPI1-capable pin (both
the PA4-7 default group and the PA15/PB3-5 remap group) already
carries another signal, with PA15 the only free pin left. Given that:

- SCLK/MOSI/MISO join the existing bit-banged SPI_CLK/SPI_IN/SPI_OUT
  bus already running from U1 to connector U$4 and POTEN_SERVO (U$6),
  as a third multi-drop leg with its own chip select - documented with
  the firmware-side bus-arbitration caveat this requires.
- CS# takes the one free pin, PA15 (TPM_CS#), with a 10k pull-up to
  +3V3 per the datasheet's recommendation for boards without a defined
  reset state (this one has no MCU reset circuit).
- VDD/GND get datasheet-recommended decoupling; NCI_VDD/NCI_GND tie to
  +3V3/GND and RST# ties to +3V3 per datasheet guidance; NC/NCI/PIRQ#/
  GPIO_00-02 are left unconnected (no spare GPIO for PIRQ#, so firmware
  polls rather than using an interrupt).

RS485-CANFD-TPM-upgrade.md is updated with the full pin audit, the
wiring rationale, and the open items this leaves for firmware/layout.
Parts:
- removed U$14: NC_MARKER, NC_MARKER:NC_MARKER
- added C39: 1u, Propio:C-EU0402
- added C40, C41, C42: 100n, Propio:C-EU0402
- added R21: 10k, Propio:R-US0402
- added U$26, U$27, U$28, U$29, U$30, U$31: NC_MARKER, NC_MARKER:NC_MARKER
- added U7: SLB9672, Propio:SLB9672
Connections:
- removed net N$9: U$14.P$1, U1.PA15
- new net N$22: U$26.P$1, U7.NC
- new net N$23: U$27.P$1, U7.NCI
- new net N$24: U$28.P$1, U7.PIRQ#
- new net N$25: U$29.P$1, U7.GPIO_00
- new net N$26: U$30.P$1, U7.GPIO_01
- new net N$27: U$31.P$1, U7.GPIO_02
- new net TPM_CS#: R21.1, U1.PA15, U7.CS#
- net +3V3: now also C39.1, C40.1, C41.1, C42.1, R21.2, U7.NCI_VDD, U7.RST#, U7.VDD
- net GND: now also C39.2, C40.2, C41.2, C42.2, U7.GND, U7.NCI_GND
- net SPI_CLK: now also U7.SCLK
- net SPI_IN: now also U7.MISO
- net SPI_OUT: now also U7.MOSI
Changed lines of the file:
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@@
 <part name="SUPPLY44" library="supply2" deviceset="GND" device=""/>
 <part name="SUPPLY45" library="supply2" deviceset="GND" device=""/>
-<part name="U$14" library="NC_MARKER" deviceset="NC_MARKER" device=""/>
 <part name="U$15" library="NC_MARKER" deviceset="NC_MARKER" device=""/>
 <part name="U$16" library="NC_MARKER" deviceset="NC_MARKER" device=""/>
@@
 <part name="+3V15" library="supply1" deviceset="+3V3" device=""/>
 <part name="+3V16" library="supply1" deviceset="+3V3" device=""/>
+<part name="U7" library="Propio" deviceset="SLB9672" device="" value="SLB9672"/>
+<part name="C39" library="Propio" deviceset="C-EU" device="0402" value="1u"/>
+<part name="C40" library="Propio" deviceset="C-EU" device="0402" value="100n"/>
+<part name="C41" library="Propio" deviceset="C-EU" device="0402" value="100n"/>
+<part name="C42" library="Propio" deviceset="C-EU" device="0402" value="100n"/>
+<part name="R21" library="Propio" deviceset="R-US" device="0402" value="10k"/>
+<part name="SUPPLY48" library="supply2" deviceset="GND" device=""/>
+<part name="+3V18" library="supply1" deviceset="+3V3" device=""/>
+<part name="+3V19" library="supply1" deviceset="+3V3" device=""/>
+<part name="+3V20" library="supply1" deviceset="+3V3" device=""/>
+<part name="U$26" library="NC_MARKER" deviceset="NC_MARKER" device=""/>
+<part name="U$27" library="NC_MARKER" deviceset="NC_MARKER" device=""/>
+<part name="U$28" library="NC_MARKER" deviceset="NC_MARKER" device=""/>
+<part name="U$29" library="NC_MARKER" deviceset="NC_MARKER" device=""/>
+<part name="U$30" library="NC_MARKER" deviceset="NC_MARKER" device=""/>
+<part name="U$31" library="NC_MARKER" deviceset="NC_MARKER" device=""/>
 </parts>
 <sheets>
@@
 <instance part="SUPPLY44" gate="GND" x="157.48" y="160.02"/>
 <instance part="SUPPLY45" gate="GND" x="157.48" y="116.84"/>
-<instance part="U$14" gate="G$1" x="-83.82" y="10.16" rot="R270"/>
 <instance part="U$15" gate="G$1" x="-129.54" y="-10.16"/>
 <instance part="U$16" gate="G$1" x="-129.54" y="-15.24"/>
@@
 </instance>
 <instance part="SUPPLY47" gate="GND" x="5.08" y="-200.66"/>
+<instance part="U7" gate="G$1" x="220" y="-130" smashed="yes">
+<attribute name="NAME" x="207.3" y="-113.49" size="1.778" layer="95"/>
+<attribute name="VALUE" x="207.3" y="-142.7" size="1.778" layer="96"/>
+</instance>
+<instance part="C39" gate="G$1" x="150" y="-150"/>
+<instance part="C40" gate="G$1" x="160" y="-150"/>
+<instance part="C41" gate="G$1" x="170" y="-150"/>
+<instance part="C42" gate="G$1" x="180" y="-150"/>
+<instance part="R21" gate="G$1" x="250" y="-125" rot="R90"/>
+<instance part="SUPPLY48" gate="GND" x="150" y="-160"/>
+<instance part="+3V18" gate="G$1" x="180" y="-118" smashed="yes">
+<attribute name="VALUE" x="182.54" y="-115.46" size="1.778" layer="96" rot="R180"/>
+</instance>
+<instance part="+3V19" gate="G$1" x="245" y="-118" smashed="yes">
+<attribute name="VALUE" x="247.54" y="-115.46" size="1.778" layer="96" rot="R180"/>
+</instance>
+<instance part="+3V20" gate="G$1" x="250" y="-115" smashed="yes">
+<attribute name="VALUE" x="252.54" y="-112.46" size="1.778" layer="96" rot="R180"/>
+</instance>
+<instance part="U$26" gate="G$1" x="192.46" y="-128.73"/>
+<instance part="U$27" gate="G$1" x="192.46" y="-131.27"/>
+<instance part="U$28" gate="G$1" x="245" y="-126.19"/>
+<instance part="U$29" gate="G$1" x="217.46" y="-110" rot="R90"/>
+<instance part="U$30" gate="G$1" x="220" y="-110" rot="R90"/>
+<instance part="U$31" gate="G$1" x="222.54" y="-110" rot="R90"/>
 </instances>
 <busses>
@@
 <label x="12.7" y="-142.24" size="1.6764" layer="94" rot="R180" xref="yes"/>
 </segment>
+<segment>
+<pinref part="U7" gate="G$1" pin="GND"/>
+<wire x1="202.22" y1="-126.19" x2="190" y2="-126.19" width="0.1524" layer="91"/>
+<wire x1="190" y1="-126.19" x2="190" y2="-152.54" width="0.1524" layer="91"/>
+<pinref part="U7" gate="G$1" pin="NCI_GND"/>
+<wire x1="202.22" y1="-136.35" x2="190" y2="-136.35" width="0.1524" layer="91"/>
+<wire x1="190" y1="-136.35" x2="190" y2="-126.19" width="0.1524" layer="91"/>
+<junction x="190" y="-126.19"/>
+<pinref part="SUPPLY48" gate="GND" pin="GND"/>
+<wire x1="150" y1="-157.46" x2="150" y2="-152.54" width="0.1524" layer="91"/>
+<pinref part="C39" gate="G$1" pin="2"/>
+<wire x1="150" y1="-152.54" x2="160" y2="-152.54" width="0.1524" layer="91"/>
+<junction x="150" y="-152.54"/>
+<pinref part="C40" gate="G$1" pin="2"/>
+<wire x1="160" y1="-152.54" x2="170" y2="-152.54" width="0.1524" layer="91"/>
+<junction x="160" y="-152.54"/>
+<pinref part="C41" gate="G$1" pin="2"/>
+<wire x1="170" y1="-152.54" x2="180" y2="-152.54" width="0.1524" layer="91"/>
+<junction x="170" y="-152.54"/>
+<pinref part="C42" gate="G$1" pin="2"/>
+<wire x1="180" y1="-152.54" x2="190" y2="-152.54" width="0.1524" layer="91"/>
+<junction x="180" y="-152.54"/>
+<junction x="190" y="-152.54"/>
+</segment>
 </net>
 <net name="+3V3" class="0">
@@
 <label x="15.24" y="-137.16" size="1.6764" layer="94" rot="R180" xref="yes"/>
 </segment>
+<segment>
+<pinref part="+3V18" gate="G$1" pin="+3V3"/>
+<wire x1="180" y1="-120.54" x2="180" y2="-123.65" width="0.1524" layer="91"/>
+<pinref part="U7" gate="G$1" pin="VDD"/>
+<wire x1="180" y1="-123.65" x2="202.22" y2="-123.65" width="0.1524" layer="91"/>
+<junction x="180" y="-123.65"/>
+<pinref part="U7" gate="G$1" pin="NCI_VDD"/>
+<wire x1="180" y1="-133.81" x2="202.22" y2="-133.81" width="0.1524" layer="91"/>
+<wire x1="180" y1="-123.65" x2="180" y2="-133.81" width="0.1524" layer="91"/>
+<junction x="180" y="-133.81"/>
+<pinref part="C42" gate="G$1" pin="1"/>
+<wire x1="180" y1="-133.81" x2="180" y2="-144.92" width="0.1524" layer="91"/>
+<pinref part="C41" gate="G$1" pin="1"/>
+<wire x1="170" y1="-144.92" x2="180" y2="-144.92" width="0.1524" layer="91"/>
+<junction x="180" y="-144.92"/>
+<pinref part="C40" gate="G$1" pin="1"/>
+<wire x1="160" y1="-144.92" x2="170" y2="-144.92" width="0.1524" layer="91"/>
+<junction x="170" y="-144.92"/>
+<pinref part="C39" gate="G$1" pin="1"/>
+<wire x1="150" y1="-144.92" x2="160" y2="-144.92" width="0.1524" layer="91"/>
+<junction x="160" y="-144.92"/>
+</segment>
+<segment>
+<pinref part="+3V19" gate="G$1" pin="+3V3"/>
+<wire x1="245" y1="-120.54" x2="245" y2="-123.65" width="0.1524" layer="91"/>
+<pinref part="U7" gate="G$1" pin="RST#"/>
+<wire x1="245" y1="-123.65" x2="237.78" y2="-123.65" width="0.1524" layer="91"/>
+</segment>
+<segment>
+<pinref part="+3V20" gate="G$1" pin="+3V3"/>
+<wire x1="250" y1="-117.54" x2="250" y2="-119.92" width="0.1524" layer="91"/>
+<pinref part="R21" gate="G$1" pin="2"/>
+</segment>
 </net>
 <net name="N$17" class="0">
@@
 <label x="142.24" y="66.04" size="2.1844" layer="94" rot="R180" xref="yes"/>
 </segment>
+<segment>
+<pinref part="U7" gate="G$1" pin="SCLK"/>
+<wire x1="237.78" y1="-128.73" x2="245" y2="-128.73" width="0.1524" layer="91"/>
+<label x="245" y="-128.73" size="2.1844" layer="94" xref="yes"/>
+</segment>
 </net>
 <net name="SPI_IN" class="0">
@@
 <label x="142.24" y="50.8" size="2.1844" layer="94" rot="R180" xref="yes"/>
 </segment>
+<segment>
+<pinref part="U7" gate="G$1" pin="MISO"/>
+<wire x1="237.78" y1="-136.35" x2="245" y2="-136.35" width="0.1524" layer="91"/>
+<label x="245" y="-136.35" size="2.1844" layer="94" xref="yes"/>
+</segment>
 </net>
 <net name="SPI_OUT" class="0">
@@
 <wire x1="266.7" y1="53.34" x2="269.24" y2="53.34" width="0.1524" layer="91"/>
 <label x="269.24" y="53.34" size="2.1844" layer="94" xref="yes"/>
+</segment>
+<segment>
+<pinref part="U7" gate="G$1" pin="MOSI"/>
+<wire x1="237.78" y1="-133.81" x2="245" y2="-133.81" width="0.1524" layer="91"/>
+<label x="245" y="-133.81" size="2.1844" layer="94" xref="yes"/>
 </segment>
 </net>
@@
 </segment>
 </net>
-<net name="N$9" class="0">
+<net name="TPM_CS#" class="0">
 <segment>
 <pinref part="U1" gate="G$1" pin="PA15"/>
-<pinref part="U$14" gate="G$1" pin="P$1"/>
+<wire x1="-83.82" y1="7.62" x2="-83.82" y2="12.7" width="0.1524" layer="91"/>
+<label x="-83.82" y="12.7" size="2.1844" layer="94" rot="R90" xref="yes"/>
+</segment>
+<segment>
+<pinref part="U7" gate="G$1" pin="CS#"/>
+<wire x1="237.78" y1="-131.27" x2="250" y2="-131.27" width="0.1524" layer="91"/>
+<wire x1="250" y1="-131.27" x2="250" y2="-130.08" width="0.1524" layer="91"/>
+<pinref part="R21" gate="G$1" pin="1"/>
+<label x="250" y="-131.27" size="2.1844" layer="94" xref="yes"/>
 </segment>
 </net>
@@
 </segment>
 </net>
+<net name="N$22" class="0">
+<segment>
+<pinref part="U7" gate="G$1" pin="NC"/>
+<pinref part="U$26" gate="G$1" pin="P$1"/>
+</segment>
+</net>
+<net name="N$23" class="0">
+<segment>
+<pinref part="U7" gate="G$1" pin="NCI"/>
+<pinref part="U$27" gate="G$1" pin="P$1"/>
+</segment>
+</net>
+<net name="N$24" class="0">
+<segment>
+<pinref part="U7" gate="G$1" pin="PIRQ#"/>
+<pinref part="U$28" gate="G$1" pin="P$1"/>
+</segment>
+</net>
+<net name="N$25" class="0">
+<segment>
+<pinref part="U7" gate="G$1" pin="GPIO_00"/>
+<pinref part="U$29" gate="G$1" pin="P$1"/>
+</segment>
+</net>
+<net name="N$26" class="0">
+<segment>
+<pinref part="U7" gate="G$1" pin="GPIO_01"/>
+<pinref part="U$30" gate="G$1" pin="P$1"/>
+</segment>
+</net>
+<net name="N$27" class="0">
+<segment>
+<pinref part="U7" gate="G$1" pin="GPIO_02"/>
+<pinref part="U$31" gate="G$1" pin="P$1"/>
+</segment>
+</net>

Commit message: Swap MCU to NXP S32K144, drop SLB9672 TPM for on-chip CSEc
U1 changes from STM32G431 to S32K144 (48-pin LQFP, no 32-pin package
exists for this family) at the schematic/netlist level: symbol and
deviceset renamed, all nets re-pinned net-for-net (pin positions kept
identical to avoid re-touching wire geometry), CAN-FD/UART/debug nets
renamed to S32K144 peripheral naming (FlexCAN0, LPUART1, SWD).

U7 (SLB9672 TPM 2.0) and its support components (decoupling, CS# pull-up,
local supply/GND instances, NC markers) are removed entirely, along with
the SLB9672 symbol/deviceset -- the S32K144's built-in CSEc hardware
security module needs no external pins or bus.

Documented in PCB/S32K144-MCU-swap.md, including an explicit flag that
CSEc is symmetric-only (AES-128/SHE) and does not cover the asymmetric
signing / post-quantum / attestation capabilities the TPM 2.0 offered --
README updated to stop claiming those. Physical LQFP48 pin numbers are
not yet mapped (the S32K1xx Data Sheet defers that to a Reference Manual
spreadsheet not available in this repo); symbol pins use functional net
names pending that lookup, same placeholder convention already used for
the other not-yet-footprinted parts on this board.
Parts:
- removed C39: 1u, Propio:C-EU0402
- removed C40, C41, C42: 100n, Propio:C-EU0402
- removed R21: 10k, Propio:R-US0402
- removed U$26, U$27, U$28, U$29, U$30, U$31: NC_MARKER, NC_MARKER:NC_MARKER
- removed U7: SLB9672, Propio:SLB9672
- U1: value STM32G431K6/K8 -> S32K144 (LQFP48); device Propio:STM32G431 -> Propio:S32K144
Connections:
- removed net FDCAN1_RX: U1.PA11, U6.RXD
- removed net FDCAN1_TX: U1.PA12, U6.TXD
- removed net N$22: U$26.P$1, U7.NC
- removed net N$23: U$27.P$1, U7.NCI
- removed net N$24: U$28.P$1, U7.PIRQ#
- removed net N$25: U$29.P$1, U7.GPIO_00
- removed net N$26: U$30.P$1, U7.GPIO_01
- removed net N$27: U$31.P$1, U7.GPIO_02
- removed net SWCLK: U$5.P$2, U1.PA14
- removed net SWDIO: U$5.P$4, U1.PA13
- removed net TPM_CS#: R21.1, U1.PA15, U7.CS#
- removed net USART1_RX: U1.PB7, U5.RxD
- removed net USART1_TX: U1.PB6, U5.TxD
- new net CAN0_RX: U1.CAN0_RX, U6.RXD
- new net CAN0_TX: U1.CAN0_TX, U6.TXD
- new net LPUART1_RX: U1.LPUART1_RX, U5.RxD
- new net LPUART1_TX: U1.LPUART1_TX, U5.TxD
- new net SWD_CLK: U$5.P$2, U1.SWD_CLK
- new net SWD_DIO: U$5.P$4, U1.SWD_DIO
- net +3V3: no longer C39.1, C40.1, C41.1, C42.1, R21.2, U7.NCI_VDD, U7.RST#, U7.VDD
- net CLK-8MHZ: now also U1.EXTAL; no longer U1.PF0-OSC_IN
- net EN-Q: now also U1.EN-Q; no longer U1.PA10
- net GND: now also U1.VSS_A; no longer C39.2, C40.2, C41.2, C42.2, U1.PB8-BOOT0, U1.VSSA, U7.GND, U7.NCI_GND
- net LED_BLUE: now also U1.LED_BLUE; no longer U1.PA5
- net LED_GREEN: now also U1.LED_GREEN; no longer U1.PA4
- net LED_RED: now also U1.LED_RED; no longer U1.PA3
- net N$10: now also U1.XTAL; no longer U1.PF1-OSC_OUT
- net N$11: now also U1.RESET_b; no longer U1.PG10-NRST
- net PWM-1: now also U1.PWM-1; no longer U1.PA8
- net PWM-2: now also U1.PWM-2; no longer U1.PB4
- net PWM-3: now also U1.PWM-3; no longer U1.PA9
- net PWM-4: now also U1.PWM-4; no longer U1.PB3
- net SEL_SERIAL: now also U1.SEL_SERIAL; no longer U1.PB5
- net SPI_CLK: now also U1.SPI_CLK; no longer U1.PA2, U7.SCLK
- net SPI_IN: now also U1.SPI_IN; no longer U1.PA0, U7.MISO
- net SPI_OUT: now also U1.SPI_OUT; no longer U1.PA1, U7.MOSI
- net VDDA-FILTRADO: now also U1.VDDA; no longer U1.VDDA/VREF+
- net V_BAT: now also U1.V_BAT; no longer U1.PB0
- net V_CORRIENTE: now also U1.V_CORRIENTE; no longer U1.PA7
- net V_TEMP: now also U1.V_TEMP; no longer U1.PA6
Other:
- note added: "S32K144 (LQFP48) @ 80MHz RUN / 112MHz HSRUN, CSEc security"
- note added: "TPM (SLB9672, U7) removed. Security now uses the S32K144's on-die CSEc (SHE-compliant hardware crypto engine) -- no external pins/bus needed. See PCB/S32K144-MCU-swap.md."
- note removed: "STM32G431K6/K8 @ up to 170MHz"

Commit message: mcu symbol
Parts:
- removed U$15, U$16: NC_MARKER, NC_MARKER:NC_MARKER
- added C39: 470n, Propio:C-EU0402
- added C40: 10n, Propio:C-EU0402
- added R21: 47K, Propio:R-US0402
- U1: value S32K144 (LQFP48) -> M0G3507QRHBRQ1; device Propio:S32K144 -> Propio:MSPM0G3507
Connections:
- removed net CAN0_RX: U1.CAN0_RX, U6.RXD
- removed net CAN0_TX: U1.CAN0_TX, U6.TXD
- removed net LPUART1_RX: U1.LPUART1_RX, U5.RxD
- removed net LPUART1_TX: U1.LPUART1_TX, U5.TxD
- removed net N$10: U$15.P$1, U1.XTAL
- removed net N$11: U$16.P$1, U1.RESET_b
- removed net SWD_CLK: U$5.P$2, U1.SWD_CLK
- removed net SWD_DIO: U$5.P$4, U1.SWD_DIO
- new net CAN_RX: U1.PA13/CAN_RX, U6.RXD
- new net CAN_TX: U1.PA12/CAN_TX, U6.TXD
- new net NRST: C40.1, R21.2, U1.NRST
- new net SWCLK: U$5.P$2, U1.PA20/SWCLK
- new net SWDIO: U$5.P$4, U1.PA19/SWDIO
- new net UART0_RX: U1.PA11/UART0_RX, U5.RxD
- new net UART0_TX: U1.PA10/UART0_TX, U5.TxD
- new net VCORE: C39.1, U1.VCORE
- net +3V3: now also R21.1, U1.VDD; no longer U1.VDD_1, U1.VDD_2
- net CLK-8MHZ: now also U1.PA6/HFCLK_IN; no longer U1.EXTAL
- net EN-Q: now also U1.PA5; no longer U1.EN-Q
- net GND: now also C39.2, C40.2, U1.PA21/VREF-, U1.PAD, U1.VSS; no longer U1.EP, U1.VSS_1, U1.VSS_2, U1.VSS_A
- net LED_BLUE: now also U1.PA7/LED_BLUE; no longer U1.LED_BLUE
- net LED_GREEN: now also U1.PA3/LED_GREEN; no longer U1.LED_GREEN
- net LED_RED: now also U1.PA0/LED_RED; no longer U1.LED_RED
- net PWM-1: now also U1.PA25/TIMA0_C1N; no longer U1.PWM-1
- net PWM-2: now also U1.PA22/TIMA0_C1; no longer U1.PWM-2
- net PWM-3: now also U1.PA24/TIMA0_C3N; no longer U1.PWM-3
- net PWM-4: now also U1.PA4/TIMA0_C3; no longer U1.PWM-4
- net SEL_SERIAL: now also U1.PA9; no longer U1.SEL_SERIAL
- net SPI_CLK: now also U1.PA17/SPI1_SCK; no longer U1.SPI_CLK
- net SPI_IN: now also U1.PA16/SPI1_POCI; no longer U1.SPI_IN
- net SPI_OUT: now also U1.PA18/SPI1_PICO; no longer U1.SPI_OUT
- net VDDA-FILTRADO: now also U1.PA23/VREF+; no longer U1.VDDA
- net V_BAT: now also U1.PA27/A0_0; no longer U1.V_BAT
- net V_CORRIENTE: now also U1.PA15/A1_0; no longer U1.V_CORRIENTE
- net V_TEMP: now also U1.PA26/A0_1; no longer U1.V_TEMP
Other:
- note added: "MCU is now TI M0G3507QRHBRQ1 (MSPM0G3507-Q1). NRST MUST be pulled to VDD (R21/C40) -- unlike the parts it replaces, this device will not leave reset otherwise. VCORE needs its own 0.47uF tank cap (C39) and must not be connected to anything else. VREF+ is fed from VDDA-FILTRADO (C4 = 1uF is the required VREF decoupling). Security: AES-128/256 + TRNG + CRC on-die, but NO SHE-class key store and NO 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"
- note added: "MSPM0G3507-Q1 (VQFN-32 RHB, 5x5mm) @ 80MHz Cortex-M0+, AEC-Q100 Grade 1"
- note removed: "S32K144 (LQFP48) @ 80MHz RUN / 112MHz HSRUN, CSEc security"
- note removed: "TPM (SLB9672, U7) removed. Security now uses the S32K144's on-die CSEc (SHE-compliant hardware crypto engine) -- no external pins/bus needed. See PCB/S32K144-MCU-swap.md."

Commit message: do the swap
Parts:
- added B7: (no value), Propio:FERRITE_BEAD_0603
- added C41: 4n7 DNP, Propio:C-EU0402
- added R22, R23: 60R4 DNP, Propio:R-US0402
- added U$26: CAN-FD IN, Propio:JST_PH-3_HOLE
- added U$27: CAN-FD OUT, Propio:JST_PH-3_HOLE
Connections:
- new net CAN_SPLIT: C41.1, R22.1, R23.2
- new net RS485_GNDISO: B7.1, C27.2, C28.2, U5.GNDISO
- net CANFD_GNDISO: now also C35.2, C36.2
- net CANFD_ISO_GND: now also C41.2, U$26.P$1, U$27.P$1; no longer C35.2, C36.2
- net CANH: now also R22.2, U$26.P$3, U$27.P$3
- net CANL: now also R23.1, U$26.P$2, U$27.P$2
- net RS485_ISO_GND: now also B7.2; no longer C27.2, C28.2
Other:
- note added: "MCU is now TI M0G3507QRHBRQ1 (MSPM0G3507-Q1). NRST MUST be pulled to VDD (R21/C40) -- unlike the parts it replaces, this device will not leave reset otherwise. VCORE needs its own 0.47uF tank cap (C39) and must not be connected to anything else. VREF+ is fed from VDDA-FILTRADO (C4 = 1uF is the required VREF decoupling). Security (TI SLAAE29A, M0G3x0x column): ROM root of trust + BIM secure boot w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"
- note added: "NEEDS: footprint/package, board placement, and a new 5V regulator for VCC (+5V_ISO_CANFD net) -- board has no 5V rail today. CAN-FD bus connectors ARE now on-sheet: U$26/U$27, JST-PH-3, deliberately 3-way so they cannot cross-mate with the 4-way RS-485 connectors (which carry +7V). R22/R23/C41 are a split termination, DO NOT POPULATE except on an end-of-bus node. See PCB/MSPM0G3507-MCU-swap.md."
- note removed: "MCU is now TI M0G3507QRHBRQ1 (MSPM0G3507-Q1). NRST MUST be pulled to VDD (R21/C40) -- unlike the parts it replaces, this device will not leave reset otherwise. VCORE needs its own 0.47uF tank cap (C39) and must not be connected to anything else. VREF+ is fed from VDDA-FILTRADO (C4 = 1uF is the required VREF decoupling). Security: AES-128/256 + TRNG + CRC on-die, but NO SHE-class key store and NO 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"
- note removed: "NEEDS: footprint/package, board placement, CANH/CANL bus connector, and a new 5V regulator for VCC (+5V_ISO_CANFD net) -- board has no 5V rail today. See PCB/RS485-CANFD-TPM-upgrade.md."
