File: PCB/LibreServo-v2.3.1.sch (EAGLE design)
At the start: 107 parts, among them M1 M1, M2 MOSFET_N+P, M3 MOSFET_N+P, M4 FAN3227/4, M5 FAN3227/4, U1 M0G3507QRHBRQ1, U10 AEAT-8800, U2 MPM3610, U3 AP2112, U4 ACS711, U5 ADM2587E, U6 ADM3055E

Commit message: 3518-q1
Parts:
- U1: value M0G3507QRHBRQ1 -> M0G3519QRHBRQ1; device Propio:MSPM0G3507 -> Propio:MSPM0G3519
Connections:
- removed net CAN_RX: U1.PA13/CAN_RX, U6.RXD
- removed net CAN_TX: U1.PA12/CAN_TX, U6.TXD
- new net CAN0_RX: U1.PA13/CAN0_RX, U6.RXD
- new net CAN0_TX: U1.PA12/CAN0_TX, U6.TXD
Other:
- note added: "MCU is now TI M0G3519QRHBRQ1 (MSPM0G3519-Q1). NRST MUST be pulled to VDD (R21/C40) -- unlike the parts it replaces, this device will not leave reset otherwise. VCORE needs its own 0.47uF tank cap (C39) and must not be connected to anything else. VREF+ is fed from VDDA-FILTRADO (C4 = 1uF is the required VREF decoupling). Security: AESADV-256 (GCM/CMAC), KEYSTORE (4 keys), CSC secure boot, flash fi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"
- note added: "MSPM0G3519-Q1 (VQFN-32 RHB, 5x5mm) @ 80MHz Cortex-M0+, 512KB/128KB, AEC-Q100 Grade 1"
- note removed: "MCU is now TI M0G3507QRHBRQ1 (MSPM0G3507-Q1). NRST MUST be pulled to VDD (R21/C40) -- unlike the parts it replaces, this device will not leave reset otherwise. VCORE needs its own 0.47uF tank cap (C39) and must not be connected to anything else. VREF+ is fed from VDDA-FILTRADO (C4 = 1uF is the required VREF decoupling). Security (TI SLAAE29A, M0G3x0x column): ROM root of trust + BIM secure boot w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"
- note removed: "MSPM0G3507-Q1 (VQFN-32 RHB, 5x5mm) @ 80MHz Cortex-M0+, AEC-Q100 Grade 1"
Changed lines of the file:
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@@
 <part name="B2" library="Propio" deviceset="FERRITE_BEAD_0603" device=""/>
 <part name="P+5" library="supply1" deviceset="+5V" device="" value="Vmot"/>
-<part name="U1" library="Propio" deviceset="MSPM0G3507" device="" value="M0G3507QRHBRQ1"/>
+<part name="U1" library="Propio" deviceset="MSPM0G3519" device="" value="M0G3519QRHBRQ1"/>
 <part name="B7" library="Propio" deviceset="FERRITE_BEAD_0603" device=""/>
 <part name="R22" library="Propio" deviceset="R-US" device="0402" value="60R4 DNP"/>
@@
 <wire x1="-60.96" y1="12.7" x2="-15.24" y2="12.7" width="0.8128" layer="94" style="shortdash"/>
 <text x="-58.42" y="40.64" size="3.81" layer="94">SWD HEADER</text>
-<text x="-195.58" y="38.1" size="5.08" layer="94">MSPM0G3507-Q1 (VQFN-32 RHB, 5x5mm) @ 80MHz Cortex-M0+, AEC-Q100 Grade 1</text>
+<text x="-195.58" y="38.1" size="5.08" layer="94">MSPM0G3519-Q1 (VQFN-32 RHB, 5x5mm) @ 80MHz Cortex-M0+, 512KB/128KB, AEC-Q100 Grade 1</text>
 <wire x1="-198.12" y1="53.34" x2="-198.12" y2="149.86" width="0.8128" layer="94" style="shortdash"/>
 <wire x1="-198.12" y1="149.86" x2="-198.12" y2="215.9" width="0.8128" layer="94" style="shortdash"/>
@@
 R22/R23/C41 are a split termination, DO NOT POPULATE except on an end-of-bus node.
 See PCB/MSPM0G3507-MCU-swap.md.</text>
-<text x="-195.58" y="-58.42" size="1.778" layer="94">MCU is now TI M0G3507QRHBRQ1 (MSPM0G3507-Q1). NRST MUST be pulled to VDD (R21/C40) -- unlike
-the parts it replaces, this device will not leave reset otherwise. VCORE needs its own 0.47uF
-tank cap (C39) and must not be connected to anything else. VREF+ is fed from VDDA-FILTRADO
-(C4 = 1uF is the required VREF decoupling).
-Security (TI SLAAE29A, M0G3x0x column): ROM root of trust + BIM secure boot with ECDSA P-256
-+ SHA-256 image authentication, AES-128/256, TRNG with self-test, permanent SWD disable.
-NO protected key store and NO hardware monotonic counter (both need CSC, absent on this die).
-See PCB/MSPM0G3507-MCU-swap.md section 6.</text>
+<text x="-195.58" y="-58.42" size="1.778" layer="94">MCU is now TI M0G3519QRHBRQ1 (MSPM0G3519-Q1). NRST MUST be pulled to VDD (R21/C40) --
+unlike the parts it replaces, this device will not leave reset otherwise. VCORE needs its own
+0.47uF tank cap (C39) and must not be connected to anything else. VREF+ is fed from
+VDDA-FILTRADO (C4 = 1uF is the required VREF decoupling). Security: AESADV-256 (GCM/CMAC),
+KEYSTORE (4 keys), CSC secure boot, flash firewalls, monotonic counter, TRNG -- this fully
+replaces the S32K144 CSEc that was dropped. See PCB/MSPM0G3519-MCU-swap.md.</text>
 </plain>
 <instances>
@@
 <attribute name="VALUE" x="43.18" y="-36.83" size="1.778" layer="96"/>
 </instance>
-<instance part="SUPPLY37" gate="GND" x="66.04" y="-63.5"/>
+<instance part="SUPPLY37" gate="GND" x="30.48" y="-44.45" rot="R270"/>
 <instance part="+3V12" gate="G$1" x="66.04" y="-15.24" smashed="yes">
 <attribute name="VALUE" x="68.58" y="-12.7" size="1.778" layer="96" rot="R180"/>
@@
 <instance part="C37" gate="G$1" x="149.86" y="-194.31"/>
 <instance part="C38" gate="G$1" x="160.02" y="-194.31"/>
-<instance part="U$24" gate="G$1" x="30.48" y="-149.86"/>
-<instance part="U$25" gate="G$1" x="91.44" y="-144.78" rot="R180"/>
+<instance part="U$24" gate="G$1" x="38.1" y="-149.86"/>
+<instance part="U$25" gate="G$1" x="83.82" y="-144.78" rot="R180"/>
 <instance part="+3V15" gate="G$1" x="93.98" y="-83.82" smashed="yes">
 <attribute name="VALUE" x="96.52" y="-81.28" size="1.778" layer="96" rot="R180"/>
@@
 <pinref part="U5" gate="G$1" pin="GND1"/>
 <pinref part="SUPPLY37" gate="GND" pin="GND"/>
-<wire x1="33.02" y1="-44.45" x2="33.02" y2="-60.96" width="0.1524" layer="91"/>
-<wire x1="33.02" y1="-60.96" x2="66.04" y2="-60.96" width="0.1524" layer="91"/>
 </segment>
 <segment>
@@
 </segment>
 </net>
-<net name="CAN_RX" class="0">
-<segment>
-<pinref part="U1" gate="G$1" pin="PA13/CAN_RX"/>
+<net name="CAN0_RX" class="0">
+<segment>
+<pinref part="U1" gate="G$1" pin="PA13/CAN0_RX"/>
 <wire x1="-76.2" y1="-15.24" x2="-71.12" y2="-15.24" width="0.1524" layer="91"/>
 <label x="-71.12" y="-15.24" size="2.1844" layer="94" xref="yes"/>
@@
 </segment>
 </net>
-<net name="CAN_TX" class="0">
-<segment>
-<pinref part="U1" gate="G$1" pin="PA12/CAN_TX"/>
+<net name="CAN0_TX" class="0">
+<segment>
+<pinref part="U1" gate="G$1" pin="PA12/CAN0_TX"/>
 <wire x1="-76.2" y1="-10.16" x2="-71.12" y2="-10.16" width="0.1524" layer="91"/>
 <label x="-71.12" y="-10.16" size="2.1844" layer="94" xref="yes"/>
@@
 <wire x1="38.1" y1="-76.2" x2="38.1" y2="-90.17" width="0.1524" layer="91"/>
 <pinref part="B4" gate="G$1" pin="1"/>
+<junction x="86.36" y="-76.2"/>
+<wire x1="86.36" y1="-76.2" x2="104.14" y2="-76.2" width="0.1524" layer="91"/>
+<wire x1="104.14" y1="-76.2" x2="104.14" y2="-88.9" width="0.1524" layer="91"/>
+<wire x1="104.14" y1="-88.9" x2="109.22" y2="-88.9" width="0.1524" layer="91"/>
 <pinref part="C27" gate="G$1" pin="1"/>
-<wire x1="109.22" y1="-88.9" x2="86.36" y2="-88.9" width="0.1524" layer="91"/>
-<wire x1="86.36" y1="-88.9" x2="86.36" y2="-76.2" width="0.1524" layer="91"/>
-<junction x="86.36" y="-76.2"/>
+<junction x="109.22" y="-88.9"/>
+<wire x1="109.22" y1="-88.9" x2="119.38" y2="-88.9" width="0.1524" layer="91"/>
 <pinref part="C28" gate="G$1" pin="1"/>
-<wire x1="119.38" y1="-88.9" x2="109.22" y2="-88.9" width="0.1524" layer="91"/>
-<junction x="109.22" y="-88.9"/>
 </segment>
 </net>
@@
 <wire x1="22.86" y1="-73.66" x2="22.86" y2="-90.17" width="0.1524" layer="91"/>
 <pinref part="B4" gate="G$1" pin="2"/>
+<junction x="93.98" y="-73.66"/>
+<wire x1="93.98" y1="-73.66" x2="124.46" y2="-73.66" width="0.1524" layer="91"/>
+<wire x1="124.46" y1="-73.66" x2="124.46" y2="-88.9" width="0.1524" layer="91"/>
+<wire x1="124.46" y1="-88.9" x2="129.54" y2="-88.9" width="0.1524" layer="91"/>
 <pinref part="C29" gate="G$1" pin="1"/>
-<wire x1="129.54" y1="-88.9" x2="93.98" y2="-88.9" width="0.1524" layer="91"/>
-<wire x1="93.98" y1="-88.9" x2="93.98" y2="-73.66" width="0.1524" layer="91"/>
-<junction x="93.98" y="-73.66"/>
+<junction x="129.54" y="-88.9"/>
+<wire x1="129.54" y1="-88.9" x2="139.7" y2="-88.9" width="0.1524" layer="91"/>
 <pinref part="C30" gate="G$1" pin="1"/>
-<wire x1="139.7" y1="-88.9" x2="129.54" y2="-88.9" width="0.1524" layer="91"/>
-<junction x="129.54" y="-88.9"/>
 </segment>
 </net>
@@
 <wire x1="97.79" y1="-134.62" x2="97.79" y2="-183.51" width="0.1524" layer="91"/>
 <junction x="97.79" y="-183.51"/>
-<wire x1="97.79" y1="-183.51" x2="139.7" y2="-183.51" width="0.1524" layer="91"/>
+<wire x1="97.79" y1="-183.51" x2="144.78" y2="-183.51" width="0.1524" layer="91"/>
+<wire x1="144.78" y1="-183.51" x2="144.78" y2="-200.66" width="0.1524" layer="91"/>
+<wire x1="144.78" y1="-200.66" x2="149.86" y2="-200.66" width="0.1524" layer="91"/>
+<junction x="149.86" y="-200.66"/>
+<wire x1="149.86" y1="-200.66" x2="149.86" y2="-196.85" width="0.1524" layer="91"/>
 <pinref part="C37" gate="G$1" pin="2"/>
-<wire x1="149.86" y1="-196.85" x2="149.86" y2="-183.51" width="0.1524" layer="91"/>
-<wire x1="149.86" y1="-183.51" x2="139.7" y2="-183.51" width="0.1524" layer="91"/>
+<wire x1="149.86" y1="-200.66" x2="160.02" y2="-200.66" width="0.1524" layer="91"/>
+<wire x1="160.02" y1="-200.66" x2="160.02" y2="-196.85" width="0.1524" layer="91"/>
 <pinref part="C38" gate="G$1" pin="2"/>
-<wire x1="160.02" y1="-196.85" x2="160.02" y2="-183.51" width="0.1524" layer="91"/>
-<wire x1="160.02" y1="-183.51" x2="149.86" y2="-183.51" width="0.1524" layer="91"/>
-<junction x="149.86" y="-183.51"/>
-</segment>
-</net>
+</segment>
+</net>

Commit message: lots of stuff
Parts:
- U1: value M0G3519QRHBRQ1 -> M0G3518QRHBRQ1; device Propio:MSPM0G3519 -> Propio:MSPM0G3518
Other:
- note added: "MCU is now TI M0G3518QRHBRQ1 (MSPM0G3518-Q1). NRST MUST be pulled to VDD (R21/C40) -- unlike the parts it replaces, this device will not leave reset otherwise. VCORE needs its own 0.47uF tank cap (C39) and must not be connected to anything else. VREF+ is fed from VDDA-FILTRADO (C4 = 1uF is the required VREF decoupling). Security: AESADV-256 (GCM/CMAC), KEYSTORE (4 keys), CSC secure boot, flash fi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"
- note added: "MSPM0G3518-Q1 (VQFN-32 RHB, 5x5mm) @ 80MHz Cortex-M0+, 256KB/128KB, AEC-Q100 Grade 1"
- note removed: "MCU is now TI M0G3519QRHBRQ1 (MSPM0G3519-Q1). NRST MUST be pulled to VDD (R21/C40) -- unlike the parts it replaces, this device will not leave reset otherwise. VCORE needs its own 0.47uF tank cap (C39) and must not be connected to anything else. VREF+ is fed from VDDA-FILTRADO (C4 = 1uF is the required VREF decoupling). Security: AESADV-256 (GCM/CMAC), KEYSTORE (4 keys), CSC secure boot, flash fi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"
- note removed: "MSPM0G3519-Q1 (VQFN-32 RHB, 5x5mm) @ 80MHz Cortex-M0+, 512KB/128KB, AEC-Q100 Grade 1"
Changed lines of the file:
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@@
 <part name="B2" library="Propio" deviceset="FERRITE_BEAD_0603" device=""/>
 <part name="P+5" library="supply1" deviceset="+5V" device="" value="Vmot"/>
-<part name="U1" library="Propio" deviceset="MSPM0G3519" device="" value="M0G3519QRHBRQ1"/>
+<part name="U1" library="Propio" deviceset="MSPM0G3518" device="" value="M0G3518QRHBRQ1"/>
 <part name="B7" library="Propio" deviceset="FERRITE_BEAD_0603" device=""/>
 <part name="R22" library="Propio" deviceset="R-US" device="0402" value="60R4 DNP"/>
@@
 <wire x1="-60.96" y1="12.7" x2="-15.24" y2="12.7" width="0.8128" layer="94" style="shortdash"/>
 <text x="-58.42" y="40.64" size="3.81" layer="94">SWD HEADER</text>
-<text x="-195.58" y="38.1" size="5.08" layer="94">MSPM0G3519-Q1 (VQFN-32 RHB, 5x5mm) @ 80MHz Cortex-M0+, 512KB/128KB, AEC-Q100 Grade 1</text>
+<text x="-195.58" y="38.1" size="5.08" layer="94">MSPM0G3518-Q1 (VQFN-32 RHB, 5x5mm) @ 80MHz Cortex-M0+, 256KB/128KB, AEC-Q100 Grade 1</text>
 <wire x1="-198.12" y1="53.34" x2="-198.12" y2="149.86" width="0.8128" layer="94" style="shortdash"/>
 <wire x1="-198.12" y1="149.86" x2="-198.12" y2="215.9" width="0.8128" layer="94" style="shortdash"/>
@@
 R22/R23/C41 are a split termination, DO NOT POPULATE except on an end-of-bus node.
 See PCB/MSPM0G3507-MCU-swap.md.</text>
-<text x="-195.58" y="-58.42" size="1.778" layer="94">MCU is now TI M0G3519QRHBRQ1 (MSPM0G3519-Q1). NRST MUST be pulled to VDD (R21/C40) --
+<text x="-195.58" y="-58.42" size="1.778" layer="94">MCU is now TI M0G3518QRHBRQ1 (MSPM0G3518-Q1). NRST MUST be pulled to VDD (R21/C40) --
 unlike the parts it replaces, this device will not leave reset otherwise. VCORE needs its own
 0.47uF tank cap (C39) and must not be connected to anything else. VREF+ is fed from
 VDDA-FILTRADO (C4 = 1uF is the required VREF decoupling). Security: AESADV-256 (GCM/CMAC),
 KEYSTORE (4 keys), CSC secure boot, flash firewalls, monotonic counter, TRNG -- this fully
-replaces the S32K144 CSEc that was dropped. See PCB/MSPM0G3519-MCU-swap.md.</text>
+replaces the S32K144 CSEc that was dropped. See PCB/MSPM0G3518-MCU-swap.md.</text>
 </plain>
 <instances>
