File: PCB/kicad/LibreServo-v4.0.0.kicad_pcb (KiCad board)
At the start: 6 copper layers, 36.5 x 42.9 mm, 84 parts, among them M1 M1, M2 MOSFET_N+P, M3 MOSFET_N+P, M4 FAN3227/4, M5 FAN3227/4, U1 STM32F301/2, U10 AEAT-8800, U2 MPM3610, U3 AP2112, U4 ACS711, U5 SIT3485

Commit message: clean up
Parts:
- B1, C1, C10, C11, C12, C13, C14, C15, C18, C19, C2, C20, C21, C3, C4, C5, C6, C9, R1, R10, R11, R12, R13, R14, R15, R16, R17, R18, R19, R2, R20, R3, R4, R5, R6, R7, R8, R9: footprint LibreServo-v2.3.1:0402 -> LibreServo-v4.0.0:0402
- B2, C16, C17, C23, C24, C7: footprint LibreServo-v2.3.1:0603 -> LibreServo-v4.0.0:0603
- C22: footprint LibreServo-v2.3.1:E2,5-6_MIN -> LibreServo-v4.0.0:E2,5-6_MIN
- C8: footprint LibreServo-v2.3.1:1206 -> LibreServo-v4.0.0:1206
- M1: footprint LibreServo-v2.3.1:SOT23 -> LibreServo-v4.0.0:SOT23
- M2, M3: footprint LibreServo-v2.3.1:DFN5X6 -> LibreServo-v4.0.0:DFN5X6
- M4, M5: footprint LibreServo-v2.3.1:MLP8 -> LibreServo-v4.0.0:MLP8
- NTC0: footprint LibreServo-v2.3.1:0402_MIN -> LibreServo-v4.0.0:0402_MIN
- RGB0: footprint LibreServo-v2.3.1:PLCC-4_2.2X2 -> LibreServo-v4.0.0:PLCC-4_2.2X2
- U$1, U$2: footprint LibreServo-v2.3.1:SERVO_SLOT -> LibreServo-v4.0.0:SERVO_SLOT
- U$100: footprint LibreServo-v2.3.1:OSC-2X1.6 -> LibreServo-v4.0.0:OSC-2X1.6
- U$3, U$4: footprint LibreServo-v2.3.1:FFC-5-0.5 -> LibreServo-v4.0.0:FFC-5-0.5
- U$5: footprint LibreServo-v2.3.1:HEADER_4_1.27_0.3 -> LibreServo-v4.0.0:HEADER_4_1.27_0.3
- U$6: footprint LibreServo-v2.3.1:POTEN_SERVO -> LibreServo-v4.0.0:POTEN_SERVO
- U$8, U$9: footprint LibreServo-v2.3.1:JST_PH-4_HOLE_B -> LibreServo-v4.0.0:JST_PH-4_HOLE_B
- U1: footprint LibreServo-v2.3.1:QFN32 -> LibreServo-v4.0.0:QFN32
- U10: footprint LibreServo-v2.3.1:QFN24 -> LibreServo-v4.0.0:QFN24
- U2: footprint LibreServo-v2.3.1:MPM36XX -> LibreServo-v4.0.0:MPM36XX
- U3: footprint LibreServo-v2.3.1:SOT25 -> LibreServo-v4.0.0:SOT25
- U4: footprint LibreServo-v2.3.1:ACS711-QFN -> LibreServo-v4.0.0:ACS711-QFN
- U5: footprint LibreServo-v2.3.1:MSOP-8 -> LibreServo-v4.0.0:MSOP-8
- UNK_HOLE_0: footprint LibreServo-v2.3.1:dummyfp0 -> LibreServo-v4.0.0:dummyfp0
- UNK_HOLE_1: footprint LibreServo-v2.3.1:dummyfp1 -> LibreServo-v4.0.0:dummyfp1
- UNK_HOLE_10: footprint LibreServo-v2.3.1:dummyfp10 -> LibreServo-v4.0.0:dummyfp10
- UNK_HOLE_11: footprint LibreServo-v2.3.1:dummyfp11 -> LibreServo-v4.0.0:dummyfp11
- UNK_HOLE_12: footprint LibreServo-v2.3.1:dummyfp12 -> LibreServo-v4.0.0:dummyfp12
- UNK_HOLE_13: footprint LibreServo-v2.3.1:dummyfp13 -> LibreServo-v4.0.0:dummyfp13
- UNK_HOLE_14: footprint LibreServo-v2.3.1:dummyfp14 -> LibreServo-v4.0.0:dummyfp14
- UNK_HOLE_15: footprint LibreServo-v2.3.1:dummyfp15 -> LibreServo-v4.0.0:dummyfp15
- UNK_HOLE_2: footprint LibreServo-v2.3.1:dummyfp2 -> LibreServo-v4.0.0:dummyfp2
- UNK_HOLE_3: footprint LibreServo-v2.3.1:dummyfp3 -> LibreServo-v4.0.0:dummyfp3
- UNK_HOLE_4: footprint LibreServo-v2.3.1:dummyfp4 -> LibreServo-v4.0.0:dummyfp4
- UNK_HOLE_5: footprint LibreServo-v2.3.1:dummyfp5 -> LibreServo-v4.0.0:dummyfp5
- UNK_HOLE_6: footprint LibreServo-v2.3.1:dummyfp6 -> LibreServo-v4.0.0:dummyfp6
- UNK_HOLE_7: footprint LibreServo-v2.3.1:dummyfp7 -> LibreServo-v4.0.0:dummyfp7
- UNK_HOLE_8: footprint LibreServo-v2.3.1:dummyfp8 -> LibreServo-v4.0.0:dummyfp8
- UNK_HOLE_9: footprint LibreServo-v2.3.1:dummyfp9 -> LibreServo-v4.0.0:dummyfp9
