File: PCB/kicad/LibreServo-v4.0.0.kicad_sch (KiCad schematic)
At the start: 95 parts, among them M1 M1, M2 MOSFET_N+P, M3 MOSFET_N+P, M4 FAN3227/4, M5 FAN3227/4, U10 AEAT-8800, U2 MPM3610, U3 AP2112, U4 ACS711

Commit message: clean up
Parts:
- added C42: 1uF, LibreServo-v4.0.0:0603, symbol LibreServo-v4.0.0-eagle-import:C-EU0603
- added C43, C44, C45: 100nF, LibreServo-v4.0.0:0402, symbol LibreServo-v4.0.0-eagle-import:C-EU0402
- added NC6, NC7: (no value), symbol LibreServo-v4.0.0-eagle-import:NC_MARKER
- added R24, R25: 10K, LibreServo-v4.0.0:0402, symbol LibreServo-v4.0.0-eagle-import:R-US0402
- added U7: SLB 9672AU2.0, Package_DFN_QFN:QFN-32-1EP_5x5mm_P0.5mm_EP3.6x3.6mm, symbol LibreServo-v4.0.0-eagle-import:SLB9672_TPM
- #U$26, #U$27: symbol LibreServo-v2.3.1-eagle-import:JST_PH-3_HOLE -> LibreServo-v4.0.0-eagle-import:JST_PH-3_HOLE
- B1: footprint LibreServo-v2.3.1:0402 -> LibreServo-v4.0.0:0402; symbol LibreServo-v2.3.1-eagle-import:FERRITE_BEAD_0402 -> LibreServo-v4.0.0-eagle-import:FERRITE_BEAD_0402
- B2, B4, B5, B6, B7: footprint LibreServo-v2.3.1:0603 -> LibreServo-v4.0.0:0603; symbol LibreServo-v2.3.1-eagle-import:FERRITE_BEAD_0603 -> LibreServo-v4.0.0-eagle-import:FERRITE_BEAD_0603
- C1, C10, C11, C12, C13, C14, C15, C18, C19, C2, C20, C21, C25, C28, C29, C3, C30, C31, C33, C34, C35, C37, C38, C39, C4, C40, C41, C5, C6, C9: footprint LibreServo-v2.3.1:0402 -> LibreServo-v4.0.0:0402; symbol LibreServo-v2.3.1-eagle-import:C-EU0402 -> LibreServo-v4.0.0-eagle-import:C-EU0402
- C16, C17, C23, C24, C26, C27, C32, C36, C7: footprint LibreServo-v2.3.1:0603 -> LibreServo-v4.0.0:0603; symbol LibreServo-v2.3.1-eagle-import:C-EU0603 -> LibreServo-v4.0.0-eagle-import:C-EU0603
- C22: footprint LibreServo-v2.3.1:E2,5-6_MIN -> LibreServo-v4.0.0:E2,5-6_MIN; symbol LibreServo-v2.3.1-eagle-import:CPOL-USE2,5-6_MIN -> LibreServo-v4.0.0-eagle-import:CPOL-USE2,5-6_MIN
- C8: footprint LibreServo-v2.3.1:1206 -> LibreServo-v4.0.0:1206; symbol LibreServo-v2.3.1-eagle-import:C-EU1206 -> LibreServo-v4.0.0-eagle-import:C-EU1206
- M1: footprint LibreServo-v2.3.1:SOT23 -> LibreServo-v4.0.0:SOT23; symbol LibreServo-v2.3.1-eagle-import:P5103EMA -> LibreServo-v4.0.0-eagle-import:P5103EMA
- M2, M3: footprint LibreServo-v2.3.1:DFN5X6 -> LibreServo-v4.0.0:DFN5X6; symbol LibreServo-v2.3.1-eagle-import:MOSFET_N+P -> LibreServo-v4.0.0-eagle-import:MOSFET_N+P
- M4, M5: footprint LibreServo-v2.3.1:MLP8 -> LibreServo-v4.0.0:MLP8; symbol LibreServo-v2.3.1-eagle-import:FAN3227/3 -> LibreServo-v4.0.0-eagle-import:FAN3227/3
- NTC0: footprint LibreServo-v2.3.1:0402_MIN -> LibreServo-v4.0.0:0402_MIN; symbol LibreServo-v2.3.1-eagle-import:R-US0402_MIN -> LibreServo-v4.0.0-eagle-import:R-US0402_MIN
- R1, R10, R11, R12, R13, R14, R15, R16, R17, R18, R19, R2, R20, R21, R22, R23, R3, R4, R5, R6, R7, R8, R9: footprint LibreServo-v2.3.1:0402 -> LibreServo-v4.0.0:0402; symbol LibreServo-v2.3.1-eagle-import:R-US0402 -> LibreServo-v4.0.0-eagle-import:R-US0402
- RGB0: footprint LibreServo-v2.3.1:PLCC-4_2.2X2 -> LibreServo-v4.0.0:PLCC-4_2.2X2; symbol LibreServo-v2.3.1-eagle-import:LED_RGB_PLCC4_2.2X2 -> LibreServo-v4.0.0-eagle-import:LED_RGB_PLCC4_2.2X2
- U$1, U$2: footprint LibreServo-v2.3.1:SERVO_SLOT -> LibreServo-v4.0.0:SERVO_SLOT; symbol LibreServo-v2.3.1-eagle-import:SLOT -> LibreServo-v4.0.0-eagle-import:SLOT
- U$100: footprint LibreServo-v2.3.1:OSC-2X1.6 -> LibreServo-v4.0.0:OSC-2X1.6; symbol LibreServo-v2.3.1-eagle-import:OSCILATOR -> LibreServo-v4.0.0-eagle-import:OSCILATOR
- U$3, U$4: footprint LibreServo-v2.3.1:FFC-5-0.5 -> LibreServo-v4.0.0:FFC-5-0.5; symbol LibreServo-v2.3.1-eagle-import:FFC-5 -> LibreServo-v4.0.0-eagle-import:FFC-5
- U$5: footprint LibreServo-v2.3.1:HEADER_4_1.27_0.3 -> LibreServo-v4.0.0:HEADER_4_1.27_0.3; symbol LibreServo-v2.3.1-eagle-import:HEADER_4_1.27_0.3 -> LibreServo-v4.0.0-eagle-import:HEADER_4_1.27_0.3
- U$6: footprint LibreServo-v2.3.1:POTEN_SERVO -> LibreServo-v4.0.0:POTEN_SERVO; symbol LibreServo-v2.3.1-eagle-import:POTEN_SERVO -> LibreServo-v4.0.0-eagle-import:POTEN_SERVO
- U$8, U$9: footprint LibreServo-v2.3.1:JST_PH-4_HOLE_B -> LibreServo-v4.0.0:JST_PH-4_HOLE_B; symbol LibreServo-v2.3.1-eagle-import:JST_PH-4_HOLEB -> LibreServo-v4.0.0-eagle-import:JST_PH-4_HOLEB
- U1: renamed from #U1; footprint (none) -> Package_DFN_QFN:Texas_RHB0032E_VQFN-32-1EP_5x5mm_P0.5mm_EP3.45x3.45mm; symbol LibreServo-v2.3.1-eagle-import:MSPM0G3519 -> LibreServo-v4.0.0-eagle-import:MSPM0G3519
- U10: footprint LibreServo-v2.3.1:QFN24 -> LibreServo-v4.0.0:QFN24; symbol LibreServo-v2.3.1-eagle-import:AEAT-8800 -> LibreServo-v4.0.0-eagle-import:AEAT-8800
- U2: footprint LibreServo-v2.3.1:MPM36XX -> LibreServo-v4.0.0:MPM36XX; symbol LibreServo-v2.3.1-eagle-import:MPM36XX -> LibreServo-v4.0.0-eagle-import:MPM36XX
- U3: footprint LibreServo-v2.3.1:SOT25 -> LibreServo-v4.0.0:SOT25; symbol LibreServo-v2.3.1-eagle-import:AP2112 -> LibreServo-v4.0.0-eagle-import:AP2112
- U4: footprint LibreServo-v2.3.1:ACS711-QFN -> LibreServo-v4.0.0:ACS711-QFN; symbol LibreServo-v2.3.1-eagle-import:ACS711 -> LibreServo-v4.0.0-eagle-import:ACS711
- U5: renamed from #U5; footprint (none) -> Package_SO:SOIC-20W_7.5x12.8mm_P1.27mm; symbol LibreServo-v2.3.1-eagle-import:ADM2587E -> LibreServo-v4.0.0-eagle-import:ADM2587E
- U6: renamed from #U6; footprint (none) -> Package_SO:SOIC-20W_7.5x12.8mm_P1.27mm; symbol LibreServo-v2.3.1-eagle-import:ADM3055E -> LibreServo-v4.0.0-eagle-import:ADM3055E
Connections:
- net +3V3: now also U1.4 (VDD), C42.1, C43.1, C44.1, C45.1, R24.2, R25.2, U7.1 (VDD), U7.14 (VDD), U7.22 (VDD), U7.8 (NCI/VDD); no longer U1.1 (VDD)
- net CAN0_RX: now also U1.17 (PA13/CAN0_RX); no longer U1.21 (PA13/CAN0_RX)
- net CAN0_TX: now also U1.16 (PA12/CAN0_TX); no longer U1.22 (PA12/CAN0_TX)
- net EN-Q: now also U1.9 (PA5); no longer U1.20 (PA5)
- net GND: now also U1.25 (PA21/VREF-), U1.5 (VSS), C42.2, C43.2, C44.2, C45.2, U7.16 (NCI/GND), U7.2 (GND), U7.23 (GND), U7.32 (GND), U7.33 (GND), U7.9 (GND); no longer U1.14 (PA21/VREF-), U1.16 (VSS)
- net LED_BLUE: now also U1.11 (PA7/LED_BLUE); no longer U1.10 (PA7/LED_BLUE)
- net LED_GREEN: now also U1.7 (PA3/LED_GREEN); no longer U1.9 (PA3/LED_GREEN)
- net LED_RED: now also U1.1 (PA0/LED_RED); no longer U1.8 (PA0/LED_RED)
- net PWM-1: now also U1.29 (PA25/TIMA0_C1N); no longer U1.18 (PA25/TIMA0_C1N)
- net PWM-2: now also U1.26 (PA22/TIMA0_C1); no longer U1.27 (PA22/TIMA0_C1)
- net PWM-3: now also U1.28 (PA24/TIMA0_C3N); no longer U1.19 (PA24/TIMA0_C3N)
- net PWM-4: now also U1.8 (PA4/TIMA0_C3); no longer U1.26 (PA4/TIMA0_C3)
- net SEL_SERIAL: now also U1.13 (PA9); no longer U1.28 (PA9)
- net SPI_CLK: now also U1.21 (PA17/SPI1_SCK), U7.19 (SCLK); no longer U1.7 (PA17/SPI1_SCK)
- net SPI_IN: now also U1.20 (PA16/SPI1_POCI), U7.24 (MISO); no longer U1.5 (PA16/SPI1_POCI)
- net SPI_OUT: now also U1.22 (PA18/SPI1_PICO), U7.21 (MOSI); no longer U1.6 (PA18/SPI1_PICO)
- net UART0_RX: now also U1.15 (PA11/UART0_RX); no longer U1.30 (PA11/UART0_RX)
- net UART0_TX: now also U1.14 (PA10/UART0_TX); no longer U1.29 (PA10/UART0_TX)
- net V_BAT: now also U1.31 (PA27/A0_0); no longer U1.13 (PA27/A0_0)
- net V_CORRIENTE: now also U1.19 (PA15/A1_0); no longer U1.12 (PA15/A1_0)
- net V_TEMP: now also U1.30 (PA26/A0_1); no longer U1.11 (PA26/A0_1)
- net at C40.1, R21.2: now also U1.3 (NRST); no longer U1.4 (NRST)
- net at B1.1, C4.1, C5.1: now also U1.27 (PA23/VREF+); no longer U1.15 (PA23/VREF+)
- net at U$100.P$3 (OUT): now also U1.10 (PA6/HFCLK_IN); no longer U1.2 (PA6/HFCLK_IN)
- net at C39.1: now also U1.32 (VCORE); no longer U1.3 (VCORE)
- new net: NC6.1 (P$1), U7.6 (NC)
- new net: NC7.1 (P$1), U7.7 (GPIO_02)
- new net TPM_CS#: R24.1, U1.6 (PA2/ROSC), U7.20 (CS#)
- new net TPM_PIRQ#: R25.1, U1.2 (PA1), U7.18 (PIRQ#)
- new net TPM_RST#: U1.18 (PA14), U7.17 (RST#)
Other:
- company: (none) -> Griffing.tech
- title: (none) -> LibreServo v4.0.0 — Griffing.tech security fork
